File: kicad_pcb/Console.kicad_pcb (KiCad board)
At the start: 2 copper layers, 218 parts, among them IC1 OPA1679, IC10 ADG1436, IC11 Opamp_Dual, IC2 OPA1641, IC3 ADG419, IC4 OPA1641, IC5 OPA1641, IC6 OPA1679, IC7 AD797

Commit message: kicad10
Parts:
- removed A-INPUT-CH1, B-INPUT-CH1, BUF-OUT-CH1, RETURN-CH1, SEND-CH1: RJ5VM, 0_Jacks:NEUTRIK_RJ5VM
- removed C15, C16, C25, C26, C27, C34, C35, C38, C42, C7, C8: 47uF, 0_Capacitors:CAP_ELEC_2.5X6.3
- removed C17, C18, C19, C20, C21, C22, C23, C24: 100pF, 0_Capacitors:0603
- removed C49, C50: 100nF, 0_Capacitors:0603
- removed C52: 220uF, 0_Capacitors:CAP_ELEC_5X10
- removed FB5, FB6, FB7, FB8: 330R@100MHz, 0_Resistors:0603
- removed IC1, IC6: OPA1679, 0_IC:SO-14
- removed IC3: ADG419, 0_IC:SO-8
- removed MIX-G1-CH1, MIX-G2-CH1, MIX-G3-CH1, MIX-MAIN-CH1, MONITOR-CH1: ~, 0_Switches:SWITCH_PUSH_7X7-POLARIZED
- removed RELAY-1: RY-[ ]W-K, 0_Switches:RELAY-RY-xW-K
- added C82: 47pF, 0_Capacitors:0603, F.Cu at (109.5, 25.5)
- added C83: 470pF, 0_Capacitors:0603, F.Cu at (109.5, 27.5)
- added C84: 470pF, 0_Capacitors:0603, F.Cu at (109.5, 29.5)
- added C85: 47pF, 0_Capacitors:0603, F.Cu at (109.5, 31.5)
- added C86: 470pF, 0_Capacitors:0603, F.Cu at (109.5, 33.5)
- added C87: 470pF, 0_Capacitors:0603, F.Cu at (109.5, 35.5)
- added C88: 47pF, 0_Capacitors:0603, F.Cu at (92.2, 35.5)
- added C89: 470pF, 0_Capacitors:0603, F.Cu at (92.2, 37.5)
- added C90: 470pF, 0_Capacitors:0603, F.Cu at (92.2, 39.5)
- added C91: 47pF, 0_Capacitors:0603, F.Cu at (92.2, 41.5)
- added C92: 470pF, 0_Capacitors:0603, F.Cu at (96.0, 25.5)
- added C93: 470pF, 0_Capacitors:0603, F.Cu at (96.0, 27.5)
- added CUE-CH1: ?-LOG, 0_Potentiometers:POTENTIOMETER-9MM, F.Cu at (61.5, 31.0)
- added FB11: 330R@100MHz, 0_Resistors:0603, F.Cu at (113.2, 29.5)
- added FB12: 330R@100MHz, 0_Resistors:0603, F.Cu at (113.2, 31.5)
- added FB13: 330R@100MHz, 0_Resistors:0603, F.Cu at (96.0, 37.5)
- added FB14: 330R@100MHz, 0_Resistors:0603, F.Cu at (96.0, 39.5)
- added R90: ~, 0_Resistors:0603, F.Cu at (61.2, 63.6)
- added R91: ~, 0_Resistors:0603, F.Cu at (61.2, 65.6)
- added R92: 75R, 0_Resistors:0603, F.Cu at (99.8, 31.5)
- added R93: 75R, 0_Resistors:0603, F.Cu at (99.8, 33.5)
- C36, C37, C53: value ~ -> 100pF
- C58, C59: value ~ -> 220pF
- IC2, IC4, IC5: value OPA1641 -> NE5532
- R31: value ~ -> 47K
- R40, R41: value 4.7K -> 2.2K
- moved C41 101.8 mm to (42.2, 59.6)
- moved C40 100.1 mm to (42.2, 57.6)
- moved C39 98.5 mm to (42.2, 55.6)
- moved R89 94.5 mm to (61.2, 61.6)
- moved ROUTE-CH1 93.7 mm to (72.9, 60.4)
- moved R61 92.1 mm to (28.4, 95.7)
- moved R62 92.1 mm to (28.4, 97.7)
- moved R63 92.1 mm to (28.4, 99.7)
- moved R64 92.1 mm to (28.4, 101.7)
- moved R35 86.3 mm to (28.4, 89.7)
- moved R36 86.3 mm to (28.4, 91.7)
- moved R37 86.3 mm to (28.4, 93.7)
- moved R31 85.2 mm to (28.4, 87.7)
- moved FB1 80.1 mm to (96.0, 29.5)
- moved FB2 80.1 mm to (96.0, 31.5)
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