File: kicad_pcb/fader.kicad_sch (KiCad schematic)
At the start: 20 parts, among them IC5 NE5532, J5 Conn_01x03

Commit message: altre cose
Parts:
- removed R63: R, 0_Resistors:0603, symbol 0_Basics:R
- removed SELECT-CH1: KS-01 green, 0_Switches:KS-01, symbol 0_ED-Sounds:SWITCH-PUSH-LED
Other:
- note added: "collegare"
- moved on the sheet: R64, REC-CH1
