File: kicad_pcb/input-jacks.kicad_sch (KiCad schematic)
At the start: 42 parts, among them IC6 OPA1679, J1 Conn_01x05

Commit message: kicad10
Parts:
- J3: value ~ -> (none)

Commit message: modifiche sostanziali al path
Parts:
- added J11: Conn_01x02, symbol Connector_Generic:Conn_01x02
- added RELAY-1: Relay, 0_Switches:FTRB3GA45ZB10, symbol 0_ED-Sounds:RELAY_AGQ210
- renumbered BUF-OUT-CH1 to OUT-CH1
Connections:
- net at C93.2, FB14.2: now also RELAY-1.3; no longer R93.1
- net at C92.1, FB13.2: now also RELAY-1.6; no longer R92.1
- net at IC6.6 (-), IC6.7, J1.2 (Pin_2): now also R92.2; no longer R93.2
- net at IC6.1, IC6.2 (-), J1.1 (Pin_1): now also R93.2; no longer R92.2
- new net: R92.1, RELAY-1.2
- new net: R93.1, RELAY-1.7
- new net: J11.1 (Pin_1), RELAY-1.4
- new net: J11.2 (Pin_2), RELAY-1.5
Other:
- note added: "collegare"
- moved on the sheet: A-INPUT-CH1, B-INPUT-CH1, C1, C10, C11, C12, C13, C14, C15, C16, C2, C3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

Commit message: fix
Parts:
- removed IC6: OPA1679, symbol Device:Opamp_Quad
- added IC1: OPA1679, 0_IC:SO-14, symbol 0_Basics:Opamp_Quad
- RELAY-1: footprint 0_Switches:FTRB3GA45ZB10 -> 0_Switches:RELAY-2FORMC
Connections:
- net +15V: now also IC1.4 (V+)
- net -15V: now also IC1.11 (V-)
- net at C15.2, R3.1: now also IC1.10 (+)
- net at J1.4 (Pin_4): now also IC1.8, IC1.9 (-)
- net at J1.2 (Pin_2), R92.2: now also IC1.6 (-), IC1.7
- net at C16.2, R4.1: now also IC1.13 (-)
- net at J1.5 (Pin_5): now also IC1.12 (+), IC1.14
- net at J1.1 (Pin_1), R93.2: now also IC1.1, IC1.2 (-)
- net at C7.2, R1.1: now also IC1.3 (+)
- net at C8.2, R2.1: now also IC1.5 (+)

Commit message: varie
Parts:
- RELAY-1: value Relay -> AGQ210A03
Connections:
- net at C16.2, R4.1: now also IC1.12 (+); no longer IC1.13 (-)
- net at IC1.14, J1.5 (Pin_5): now also IC1.13 (-); no longer IC1.12 (+)
Changed lines of the file:
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@@
 	(wire
 		(pts
+			(xy 147.32 148.59) (xy 162.56 148.59)
+		)
+		(stroke
+			(width 0)
+			(type default)
+		)
+	)
+	(wire
+		(pts
 			(xy 143.51 143.51) (xy 147.32 143.51)
 		)
@@
 	(wire
 		(pts
-			(xy 147.32 148.59) (xy 162.56 148.59)
-		)
-		(stroke
-			(width 0)
-			(type default)
-		)
-	)
-	(wire
-		(pts
 			(xy 104.14 146.05) (xy 104.14 140.97)
 		)
@@
 			)
 		)
-		(property "Value" "Relay"
+		(property "Value" "AGQ210A03"
 			(at 143.51 34.544 0)
 			(show_name no)
@@
 		(lib_id "0_Basics:Opamp_Quad")
 		(at 154.94 156.21 0)
+		(mirror x)
 		(unit 4)
 		(body_style 1)
@@
 		(dnp no)
 		(property "Reference" "IC1"
-			(at 150.368 155.702 0)
+			(at 150.368 156.718 0)
 			(show_name no)
 			(do_not_autoplace yes)
@@
 		)
 		(property "Value" "OPA1679"
-			(at 150.368 156.972 0)
+			(at 150.368 155.448 0)
 			(show_name no)
 			(do_not_autoplace yes)
