File: kicad_pcb/appunti.kicad_sch (KiCad schematic)
At the start: 55 parts, among them IC10 ADG1436, IC11 Opamp_Dual, IC7 AD797

Commit message: kicad10
Parts:
- removed IC10: ADG1436, 0_IC:TSSOP-16, symbol 0_ED-Sounds:ADG1436
- C63, C64, C68, C69, C71, IC8, IC9, R65, SW-LEFT-1, SW-RIGHT-1: value ~ -> (none)

Commit message: fix varie
Parts:
- added unit 1 of BLEND1
Connections:
- net GND: now also BLEND1.2 (WIPER); no longer BLEND1.2 (WIPER)
- net at R70.1, R71.2: now also BLEND1.1 (CCW); no longer BLEND1.1 (CCW)
- net at R68.2, R69.1: now also BLEND1.3 (CW); no longer BLEND1.3 (CW)
Other:
- moved on the sheet: BLEND1B
Changed lines of the file:
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@@
+	(symbol
+		(lib_id "0_ED-Sounds:POTENTIOMETER_DUAL")
+		(at 156.21 123.19 0)
+		(unit 2)
+		(body_style 1)
+		(exclude_from_sim no)
+		(in_bom yes)
+		(on_board yes)
+		(in_pos_files yes)
+		(dnp no)
+		(fields_autoplaced yes)
+		(property "Reference" "BLEND1"
+			(at 151.384 128.2954 90)
+			(show_name no)
+			(do_not_autoplace yes)
+			(effects
+				(font
+					(size 1.016 1.016)
+					(thickness 0.127)
+				)
+				(justify left)
+			)
+		)
+		(property "Value" "10K-LIN"
+			(at 153.162 128.27 90)
+			(show_name no)
+			(do_not_autoplace yes)
+			(effects
+				(font
+					(size 0.889 0.889)
+				)
+				(justify left bottom)
+			)
+		)
+		(property "Footprint" "0_Potentiometers:POTENTIOMETER-9MM"
+			(at 156.21 120.396 0)
+			(hide yes)
+			(show_name no)
+			(do_not_autoplace no)
+			(effects
+				(font
+					(size 1.27 1.27)
+				)
+			)
+		)
+		(property "Datasheet" ""
+			(at 156.21 123.19 0)
+			(hide yes)
+			(show_name no)
+			(do_not_autoplace no)
+			(effects
+				(font
+					(size 1.27 1.27)
+				)
+			)
+		)
+		(property "Description" "Resistor (variable)"
+			(at 156.718 118.364 0)
+			(hide yes)
+			(show_name no)
+			(do_not_autoplace no)
+			(effects
+				(font
+					(size 1.27 1.27)
+				)
+			)
+		)
+		(property "Sim.Device" "R"
+			(at 156.21 123.19 0)
+			(hide yes)
+			(show_name no)
+			(do_not_autoplace no)
+			(effects
+				(font
+					(size 1.27 1.27)
+				)
+			)
+		)
+		(property "Sim.Type" "POT"
+			(at 156.21 123.19 0)
+			(hide yes)
+			(show_name no)
+			(do_not_autoplace no)
+			(effects
+				(font
+					(size 1.27 1.27)
+				)
+			)
+		)
+		(property "Sim.Pins" "1=r0 2=wiper 3=r1"
+			(at 156.21 123.19 0)
+			(hide yes)
+			(show_name no)
+			(do_not_autoplace no)
+			(effects
+				(font
+					(size 1.27 1.27)
+				)
+			)
+		)
+		(property "Sim.Params" "r=\"\""
+			(at 156.21 123.19 0)
+			(hide yes)
+			(show_name no)
+			(do_not_autoplace no)
+			(effects
+				(font
+					(size 1.27 1.27)
+				)
+			)
+		)
+		(pin "4"
+		)
+		(pin "5"
+		)
+		(pin "6"
+		)
+		(pin "1"
+		)
+		(pin "2"
+		)
+		(pin "3"
+		)
+		(instances
+			(project "Console"
+				(path "/1fbbd2a3-bb57-473e-beb7-4110a7f2d116/b833796d-8766-4e88-a7f0-c319ee501070"
+					(reference "BLEND1")
+					(unit 2)
+				)
+			)
+		)
+	)
 	(symbol
 		(lib_id "0_ED-Sounds:POTENTIOMETER_DUAL")
