File: kicad_pcb/mono_channel.kicad_sch (KiCad schematic)
At the start: 108 parts, among them IC1 OPA1679, IC2 NE5532, IC3 ADG419, IC4 NE5532, J10 Conn_01x02, J11 Conn_01x02, J2 Conn_01x05, J4 Conn_01x02, J6 Conn_01x03, J8 Conn_01x05

Commit message: kicad10
Parts:
- removed C49, C50: 100nF, 0_Capacitors:0603, symbol 0_Basics:C
- removed IC3: ADG419, symbol 0_ED-Sounds:ADG419
- removed MONITOR-CH1: ~, 0_Switches:SWITCH_PUSH_7X7-POLARIZED, symbol 0_ED-Sounds:SWITCH-PUSH-LATCHING
- removed RELAY-1: RY-[ ]W-K, 0_Switches:RELAY-RY-xW-K, symbol 0_ED-Sounds:RELAY-DPDT
- added RELAY-2, RELAY-3, RELAY-4: AGQ210A03, 0_Switches:FTRB3GA45ZB10, symbol 0_ED-Sounds:RELAY_AGQ210
- HPF-CH1, INSERT-CH1, J9, PFL-CH1, R44, R45, R46, R47, R48, R49, R50, R51, R52, R53, R54, R55, R56, R57, R58, R59, R90, R91, ROUTE-CH1: value ~ -> (none)
Connections:
- no-connect marks 4 -> 3
Other:
- note added: "CAPIRE COME"
- note removed: "claude dice GND deve essere digitale, anche per i caps?"
- note removed: "devo misurare quali sono i pin NC veramente quando è alimentato"
- moved on the sheet: AUX1-CH1A, AUX1-CH1B, AUX2-CH1A, AUX2-CH1B, AUX3-CH1A, AUX3-CH1B, AUX4-CH1A, AUX4-CH1B, C27, C34, C35, C36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

Commit message: modifiche sostanziali al path
Parts:
- removed J11: Conn_01x02, symbol Connector_Generic:Conn_01x02
- removed R89: 75R, 0_Resistors:0603, symbol 0_Basics:R
- added DIR/PROC-CH1, OUT-PRE/POST-CH1: (no value), 0_Switches:SWITCH_PUSH_7X7-POLARIZED, symbol 0_ED-Sounds:SWITCH-PUSH-LATCHING
- added LED-OUT-DIR-CH1, LED-OUT-DIR-CH2, LED-OUT-PROC-CH1, LED-OUT-PROC-CH2: orange, 0_Leds:LED3MM, symbol 0_Basics:LED
- added R100, R101, R98, R99: R, 0_Resistors:0603, symbol 0_Basics:R
- added R102, R96, R97: 75R, 0_Resistors:0603, symbol 0_Basics:R
- added R94, R95: (no value), 0_Resistors:0603, symbol 0_Basics:R
Connections:
- net +5VD is gone; now on net VD: HPF-CH1.2-C (C), INSERT-CH1.2-C (C), J4.1 (Pin_1), PFL-CH1.2-C (C)
- net GND: now also RELAY-2.3, RELAY-3.2, RELAY-3.7, R96.1; no longer J10.2 (Pin_2)
- net GNDD: now also DIR/PROC-CH1.1-NC (NC), R100.2, R101.2, R98.2, R99.2
- net at C25.2, R9.1: now also RELAY-4.5
- net at C39.1, HPF-CH1.1-NC (NC): now also RELAY-4.6
- net at INSERT-CH1.1-C (C), R27.1: now also RELAY-2.6, R97.2
- net at C58.2, IC4.1, R38.1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: now also R94.2
- net at AUX1-CH1.3 (CW), AUX2-CH1.3 (CW), AUX3-CH1.3 (CW)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: now also RELAY-2.4, RELAY-2.7
- net at AUX1-CH1.6 (CW), AUX2-CH1.6 (CW), AUX3-CH1.6 (CW)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: now also R102.2
- net at RELAY-3.3: now also R95.1
- net BUS-AFL-RIGHT: now reaches RELAY-3.4
- net BUS-AFL-LEFT: now reaches RELAY-3.5
- net at RELAY-3.6: now also R94.1
- net at LED-MONITOR-B-CH1.2 (A): now also RELAY-4.2
- net VD: now reaches RELAY-4.3
- net VD: now also DIR/PROC-CH1.1-NO (NO), DIR/PROC-CH1.2-C (C), OUT-PRE/POST-CH1.2-C (C)
- net at RELAY-4.4: now also LED-MONITOR-A-CH1.2 (A)
- net at RELAY-4.7: now also C26.2, R16.1
- net at J10.1 (Pin_1): now also R96.2
- net at C59.2, IC4.7, R39.1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: now also R95.2
- new net: LED-OUT-PROC-CH1.1 (K), R98.1
- new net: J10.2 (Pin_2), OUT-PRE/POST-CH1.1-C (C)
- new net: OUT-PRE/POST-CH1.1-NC (NC), R97.1
- new net: OUT-PRE/POST-CH1.1-NO (NO), R102.1
- new net: LED-OUT-PROC-CH2.1 (K), R101.1
- new net: LED-OUT-DIR-CH1.1 (K), R99.1
- new net: DIR/PROC-CH1.2-NC (NC), LED-OUT-DIR-CH1.2 (A)
- new net: DIR/PROC-CH1.2-NO (NO), LED-OUT-PROC-CH1.2 (A)
- new net: LED-OUT-PROC-CH2.2 (A), OUT-PRE/POST-CH1.2-NO (NO)
- new net: LED-OUT-DIR-CH2.1 (K), R100.1
- new net: LED-OUT-DIR-CH2.2 (A), OUT-PRE/POST-CH1.2-NC (NC)
- no-connect marks 3 -> 5
Other:
- note added: "bisognerebbe fare mirror del postfader"
- note added: "collegare"
- note removed: "CAPIRE COME"
- note removed: "afl con relay"
- note removed: "capire se unico connettore"
- note removed: "coppia di opamp che isola"
- note removed: "dopo il routing valutare se posso metterne altre in parallelo"
- note removed: "metering in routing capire se meglio unico connettore da 6 o 8"
- note removed: "postfade output stereo oppure mono prima del pan"
- moved on the sheet: AUX1-CH1A, AUX1-CH1B, AUX2-CH1A, AUX2-CH1B, AUX3-CH1A, AUX3-CH1B, AUX4-CH1A, AUX4-CH1B, C25, C26, C27, C34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

Commit message: altre cose
Parts:
- added MON/MIX-CH1: (no value), 0_Switches:SWITCH_PUSH_7X7-POLARIZED, symbol 0_ED-Sounds:SWITCH-PUSH-LATCHING
Connections:
- net GNDD: now also MON/MIX-CH1.1-NC (NC), MON/MIX-CH1.2-NC (NC)
- net VD: now also MON/MIX-CH1.1-NO (NO), MON/MIX-CH1.2-NO (NO)
- new net: MON/MIX-CH1.1-C (C), MON/MIX-CH1.2-C (C)
Other:
- moved on the sheet: DIR/PROC-CH1A, DIR/PROC-CH1B, LED-OUT-DIR-CH1, LED-OUT-PROC-CH1, R102, R98, R99

Commit message: fx bypass
Parts:
- added FX-FOLLOW-A-CH1, FX-FOLLOW-B-CH1, FX-FOLLOW-PATH-CH1: orange, 0_Leds:LED3MM, symbol 0_Basics:LED
- added FX-FOLLOW-CH1: (no value), 0_Switches:SWITCH_PUSH_7X7-POLARIZED, symbol 0_ED-Sounds:SWITCH-PUSH-LATCHING
- added R103, R104, R106: R, 0_Resistors:0603, symbol 0_Basics:R
- added RELAY-5: AGQ210A03, 0_Switches:FTRB3GA45ZB10, symbol 0_ED-Sounds:RELAY_AGQ210
Connections:
- net GNDD: now also FX-FOLLOW-CH1.1-NC (NC), FX-FOLLOW-CH1.2-NC (NC), R103.2, R104.2, R106.2
- net VD: now also FX-FOLLOW-CH1.1-NO (NO), FX-FOLLOW-CH1.2-NO (NO)
- net at C39.1, HPF-CH1.1-NC (NC): now also RELAY-5.5; no longer RELAY-4.6
- net at R27.1, R97.2, RELAY-2.6: now also RELAY-5.3; no longer INSERT-CH1.1-C (C)
- new net: FX-FOLLOW-CH1.1-C (C), FX-FOLLOW-CH1.2-C (C)
- new net: FX-FOLLOW-A-CH1.1 (K), R106.1
- new net: RELAY-4.6, RELAY-5.6
- new net: INSERT-CH1.1-C (C), RELAY-5.4
- new net: FX-FOLLOW-B-CH1.1 (K), R104.1
- new net: FX-FOLLOW-PATH-CH1.1 (K), R103.1
- new net: RELAY-5.2, RELAY-5.7
Other:
- note added: "bisognerebbe fare mirror del postfader unico modo togliere i led"
- note removed: "bisognerebbe fare mirror del postfader"
- moved on the sheet: C25, C26, C27, C34, C35, C36, C37, C38, C39, C40, C41, C42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

Commit message: metering
Parts:
- removed R102, R97: 75R, 0_Resistors:0603, symbol 0_Basics:R
- added C97, C98: 100nF, 0_Capacitors:0603, symbol 0_Basics:C
- added IC10: NE5532, 0_IC:SO-8, symbol 0_Basics:Opamp_Dual
- added J12: Conn_01x02, symbol Connector_Generic:Conn_01x02
- added R105, R63, R89: 75R, 0_Resistors:0603, symbol 0_Basics:R
Connections:
- net +15V: now also C98.1, IC10.8 (V+)
- net -15V: now also C97.2, IC10.4 (V-)
- net GND: now also C97.1, C98.2
- net VD: no longer RELAY-4.3
- net at C25.2, R9.1, RELAY-4.5: now also RELAY-4.2
- net at R27.1, RELAY-2.6, RELAY-5.3: now also OUT-PRE/POST-CH1.1-NC (NC), IC10.5 (+)
- net at OUT-PRE/POST-CH1.1-C (C): now also R105.1; no longer J10.2 (Pin_2)
- net at AUX1-CH1.6 (CW), AUX2-CH1.6 (CW), AUX3-CH1.6 (CW)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: now also OUT-PRE/POST-CH1.1-NO (NO)
- net at LED-MONITOR-B-CH1.2 (A): no longer RELAY-4.2
- net at LED-MONITOR-A-CH1.2 (A): no longer RELAY-4.4
- net at C26.2, R16.1, RELAY-4.7: now also RELAY-4.4
- new net: IC10.1, IC10.2 (-), R63.2
- new net: IC10.3 (+), RELAY-4.3
- new net: IC10.6 (-), IC10.7, R89.2
- new net: J10.2 (Pin_2), R105.2
- new net: J12.1 (Pin_1), R63.1
- new net: J12.2 (Pin_2), R89.1
Other:
- note added: "serve GND?"
- moved on the sheet: C25, C26, FX-FOLLOW-A-CH1, FX-FOLLOW-B-CH1, FX-FOLLOW-PATH-CH1, GAIN-A-CH1, GAIN-B-CH1, IC1A, IC1B, IC1C, IC1D, J2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

Commit message: fix
Parts:
- RELAY-2, RELAY-3, RELAY-4, RELAY-5: footprint 0_Switches:FTRB3GA45ZB10 -> 0_Switches:RELAY-2FORMC
Connections:
- net +15V: no longer IC1.4 (V+)
- net -15V: no longer IC1.11 (V-)
Changed lines of the file:
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@@
 			)
 		)
-		(property "Footprint" "0_Switches:FTRB3GA45ZB10"
+		(property "Footprint" "0_Switches:RELAY-2FORMC"
 			(at 368.554 193.548 0)
 			(hide yes)
@@
 			)
 		)
-		(property "Footprint" "0_Switches:FTRB3GA45ZB10"
+		(property "Footprint" "0_Switches:RELAY-2FORMC"
 			(at 128.016 164.338 0)
 			(hide yes)
@@
 			)
 		)
-		(property "Footprint" "0_Switches:FTRB3GA45ZB10"
+		(property "Footprint" "0_Switches:RELAY-2FORMC"
 			(at 148.844 164.338 0)
 			(hide yes)
@@
 			)
 		)
-		(property "Footprint" "0_Switches:FTRB3GA45ZB10"
+		(property "Footprint" "0_Switches:RELAY-2FORMC"
 			(at 239.014 145.288 0)
 			(hide yes)

Commit message: varie
Parts:
- removed C58, C59: 220pF, 0_Capacitors:0603, symbol 0_Basics:C
- removed IC1: OPA1679, symbol Device:Opamp_Quad
- added IC3: OPA1679, 0_IC:SO-14, symbol 0_Basics:Opamp_Quad
- IC10: value NE5532 -> TL072
Connections:
- net +15V: now also IC3.4 (V+)
- net -15V: now also IC3.11 (V-)
- net GND: now also IC3.10 (+), IC3.12 (+), IC3.3 (+), IC3.5 (+)
- net at C26.1, R15.1: now also IC3.14
- net at R6.1, R7.2: now also IC3.1
- net at R5.1, R6.2: now also IC3.2 (-)
- net at RELAY-4.3 (COM2): now also IC10.5 (+); no longer IC10.3 (+)
- net at OUT-PRE/POST-CH1.1-NC (NC), R27.1, RELAY-2.6 (COM1)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: now also IC10.3 (+); no longer IC10.5 (+)
- net at C25.1, R8.1: now also IC3.7
- net at GAIN-A-CH1.1, R10.1, R7.1: now also IC3.6 (-)
- net at R11.1, R12.2: now also IC3.9 (-)
- net at GAIN-B-CH1.1, R13.1, R14.1: now also IC3.13 (-)
- net at R12.1, R13.2: now also IC3.8
- new net: IC10.6 (-), IC10.7, R63.2
- new net: IC10.1, IC10.2 (-), R89.2
Other:
- moved on the sheet: RELAY-2

Commit message: fix varie
Parts:
- removed LED-OUT-PROC-CH1: orange, 0_Leds:LED3MM, symbol 0_Basics:LED
- removed R98: R, 0_Resistors:0603, symbol 0_Basics:R
- renumbered LED-OUT-DIR-CH2 to LED-OUT-PRE-CH2, LED-MONITOR-A-CH1 to LED-SOURCE-A-CH1, LED-MONITOR-B-CH1 to LED-SOURCE-B-CH1, MON/MIX-CH1 to SOURCE-CH1
Connections:
- net VD: no longer OUT-PRE/POST-CH1.2-C (C)
- net at DIR/PROC-CH1.2-NO (NO): now also OUT-PRE/POST-CH1.2-C (C)
- net BUS_PFL renamed BUS-PFL
Other:
- note added: "collegare magari diretto al relay"
- moved on the sheet: DIR/PROC-CH1A, DIR/PROC-CH1B, LED-OUT-DIR-CH1, LED-OUT-PRE-CH2, LED-OUT-PROC-CH2, R100, R101, R99
