File: kicad_pcb/mono_channel.kicad_sch (KiCad schematic)
At the start: 129 parts, among them IC10 TL072, IC2 NE5532, IC3 OPA1679, IC4 NE5532, J10 Conn_01x02, J12 Conn_01x02, J2 Conn_01x05, J4 Conn_01x02, J6 Conn_01x03, J8 Conn_01x05

Commit message: altro
Other:
- note added: "non serve pilotarlo su MCU, basta mandarlo su quella pcb ma va diretto al h bridge senza passare per mcu"
- note removed: "collegare magari diretto al relay"
Changed lines of the file:
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@@
 		)
 	)
-	(text "collegare\nmagari diretto al relay"
+	(text "non serve pilotarlo\nsu MCU, basta mandarlo\nsu quella pcb ma va diretto\nal h bridge senza passare\nper mcu"
 		(exclude_from_sim no)
 		(at 105.41 35.56 0)
